File: exa_tim.sch (KiCad schematic (older format))
At the start: 54 parts, among them J1 Conn_ARM_JTAG_SWD_10, J2 FH12A-24S-0.5SH(55), Q1 SI2333DS-T1-E3, Q2 DMN3067LW-7, SW1 SKHLLFA010, SW2 SKHLLFA010, SW3 SKHLLFA010, SW4 SKHLLFA010, U1 STM32L071KZUx, U2 CAM-M8Q-0, Y1 9HT11-32.768KDZF-T

Commit message: General cleanup
Parts:
- BT1: Notice CR2032 -> CR2450
- C5: footprint Resistor_SMD:R_0603_1608Metric -> Capacitor_SMD:C_0603_1608Metric
- D1: value LED_ALT -> LTST-C194KSKT
- LS1: value Speaker -> CUI_CSS-0575A-SMT
- R1, R4, R7: value 1M -> 100k
- R8: value 3R -> 3
Changed lines of the file:
@@
 P 2050 2000
 F 0 "R1" V 2150 1950 50  0000 L CNN
-F 1 "1M" V 1950 1950 50  0000 L CNN
+F 1 "100k" V 1950 1950 50  0000 L CNN
 F 2 "Resistor_SMD:R_0603_1608Metric" V 1980 2000 50  0001 C CNN
 F 3 "~" H 2050 2000 50  0001 C CNN
@@
 F 2 "exa_tim:NL5077-LF" V 900 4210 50  0001 C CNN
 F 3 "~" V 900 4210 50  0001 C CNN
-F 4 "CR2032" H 900 4150 50  0001 C CNN "Notice"
+F 4 "CR2450" H 900 4150 50  0001 C CNN "Notice"
 	1    900  4150
 	1    0    0    -1
@@
 P 9150 5850
 F 0 "R7" H 9220 5896 50  0000 L CNN
-F 1 "1M" H 9220 5805 50  0000 L CNN
+F 1 "100k" H 9220 5805 50  0000 L CNN
 F 2 "Resistor_SMD:R_0603_1608Metric" V 9080 5850 50  0001 C CNN
 F 3 "~" H 9150 5850 50  0001 C CNN
@@
 P 9550 5850
 F 0 "R8" H 9620 5896 50  0000 L CNN
-F 1 "3R" H 9620 5805 50  0000 L CNN
+F 1 "3" H 9620 5805 50  0000 L CNN
 F 2 "Resistor_SMD:R_0603_1608Metric" V 9480 5850 50  0001 C CNN
 F 3 "~" H 9550 5850 50  0001 C CNN
@@
 P 5300 2950
 F 0 "R4" H 5370 2996 50  0000 L CNN
-F 1 "1M" H 5370 2905 50  0000 L CNN
+F 1 "100k" H 5370 2905 50  0000 L CNN
 F 2 "Resistor_SMD:R_0603_1608Metric" V 5230 2950 50  0001 C CNN
 F 3 "~" H 5300 2950 50  0001 C CNN
@@
 P 2750 4600
 F 0 "D1" H 2742 4345 50  0000 C CNN
-F 1 "LED_ALT" H 2742 4436 50  0000 C CNN
+F 1 "LTST-C194KSKT" H 2742 4436 50  0000 C CNN
 F 2 "LED_SMD:LED_0603_1608Metric" H 2750 4600 50  0001 C CNN
 F 3 "~" H 2750 4600 50  0001 C CNN
@@
 P 3000 5150
 F 0 "LS1" H 3170 5146 50  0000 L CNN
-F 1 "Speaker" H 3170 5055 50  0000 L CNN
+F 1 "CUI_CSS-0575A-SMT" H 3170 5055 50  0000 L CNN
 F 2 "exa_tim:CUI_CSS-0575A-SMT" H 3000 4950 50  0001 C CNN
 F 3 "~" H 2990 5100 50  0001 C CNN
@@
 F 0 "C5" V 2002 1800 50  0000 C CNN
 F 1 "100nF" V 1911 1800 50  0000 C CNN
-F 2 "Resistor_SMD:R_0603_1608Metric" H 1788 1650 50  0001 C CNN
+F 2 "Capacitor_SMD:C_0603_1608Metric" H 1788 1650 50  0001 C CNN
 F 3 "~" H 1750 1800 50  0001 C CNN
 	1    1750 1800

Commit message: Rework GND plane, power distrubution and PU
PU are now 1M ohm. GND is the only power plane.
Parts:
- BT1: Notice CR2450 -> CR2450 or CR2477
- J1: footprint Connector_PinHeader_1.27mm:PinHeader_2x05_P1.27mm_Horizontal -> Connector_PinHeader_1.27mm:PinHeader_2x05_P1.27mm_Vertical_SMD
- R1, R4, R7: value 100k -> 1M
Changed lines of the file:
@@
 P 2050 2000
 F 0 "R1" V 2150 1950 50  0000 L CNN
-F 1 "100k" V 1950 1950 50  0000 L CNN
+F 1 "1M" V 1950 1950 50  0000 L CNN
 F 2 "Resistor_SMD:R_0603_1608Metric" V 1980 2000 50  0001 C CNN
 F 3 "~" H 2050 2000 50  0001 C CNN
@@
 F 2 "exa_tim:NL5077-LF" V 900 4210 50  0001 C CNN
 F 3 "~" V 900 4210 50  0001 C CNN
-F 4 "CR2450" H 900 4150 50  0001 C CNN "Notice"
+F 4 "CR2450 or CR2477" H 900 4150 50  0001 C CNN "Notice"
 	1    900  4150
 	1    0    0    -1
@@
 P 9150 5850
 F 0 "R7" H 9220 5896 50  0000 L CNN
-F 1 "100k" H 9220 5805 50  0000 L CNN
+F 1 "1M" H 9220 5805 50  0000 L CNN
 F 2 "Resistor_SMD:R_0603_1608Metric" V 9080 5850 50  0001 C CNN
 F 3 "~" H 9150 5850 50  0001 C CNN
@@
 F 0 "J1" H 1910 6496 50  0000 R CNN
 F 1 "Conn_ARM_JTAG_SWD_10" H 1910 6405 50  0000 R CNN
-F 2 "Connector_PinHeader_1.27mm:PinHeader_2x05_P1.27mm_Horizontal" H 2400 5900 50  0001 L TNN
+F 2 "Connector_PinHeader_1.27mm:PinHeader_2x05_P1.27mm_Vertical_SMD" H 2400 5900 50  0001 L TNN
 F 3 "http://infocenter.arm.com/help/topic/com.arm.doc.faqs/attached/13634/cortex_debug_connectors.pdf" V 2000 5200 50  0001 C CNN
 	1    2350 6450
@@
 P 5300 2950
 F 0 "R4" H 5370 2996 50  0000 L CNN
-F 1 "100k" H 5370 2905 50  0000 L CNN
+F 1 "1M" H 5370 2905 50  0000 L CNN
 F 2 "Resistor_SMD:R_0603_1608Metric" V 5230 2950 50  0001 C CNN
 F 3 "~" H 5300 2950 50  0001 C CNN

Commit message: Added 3d models and moved some parts for fitting
The 3d models are not licenced under the permissive licensce.
They come from their manufacturer and some other free sources.
Parts:
- J2: footprint Connector_FFC-FPC:Hirose_FH12-24S-0.5SH_1x24-1MP_P0.50mm_Horizontal -> exa_tim:Hirose_FH12-24S-0.5SH_1x24-1MP_P0.50mm_Horizontal
- L1: footprint Inductor_SMD:L_Coilcraft_LPS4018 -> exa_tim:L_Coilcraft_LPS4018
- U2: value CAM-M8Q-0 -> CAM-M8C-0
Changed lines of the file:
@@
 F 0 "J2" H 10769 625 50  0000 C CNN
 F 1 "FH12A-24S-0.5SH(55)" H 10769 716 50  0000 C CNN
-F 2 "Connector_FFC-FPC:Hirose_FH12-24S-0.5SH_1x24-1MP_P0.50mm_Horizontal" H 10850 2050 50  0001 C CNN
+F 2 "exa_tim:Hirose_FH12-24S-0.5SH_1x24-1MP_P0.50mm_Horizontal" H 10850 2050 50  0001 C CNN
 F 3 "https://www.mouser.de/datasheet/2/185/FH12_catalog-939276.pdf" H 10850 2050 50  0001 C CNN
 	1    10850 2050
@@
 F 0 "L1" V 9275 4850 50  0000 C CNN
 F 1 "LPS4018-683MRB" V 9184 4850 50  0000 C CNN
-F 2 "Inductor_SMD:L_Coilcraft_LPS4018" H 9050 4850 50  0001 C CNN
+F 2 "exa_tim:L_Coilcraft_LPS4018" H 9050 4850 50  0001 C CNN
 F 3 "https://www.mouser.de/datasheet/2/597/lps4018-270702.pdf" H 9050 4850 50  0001 C CNN
 	1    9050 4850
@@
 P 6350 1800
 F 0 "U2" H 6350 2667 50  0000 C CNN
-F 1 "CAM-M8Q-0" H 6350 2576 50  0000 C CNN
+F 1 "CAM-M8C-0" H 6350 2576 50  0000 C CNN
 F 2 "exa_tim:LCC100P960X1400X210-31N" H 5800 800 50  0001 L BNN
 F 3 "" H 5450 900 50  0001 L BNN

Commit message: Changed epaper connection to bottom feeding
Switched from FH12A to FH12, which is bottom feeding. This way the
PCB doesn't need to be mounted with the top facing down.

Also moved the battery now back to the original version. Hopefully
the battery will fit properly.
Parts:
- J2: value FH12A-24S-0.5SH(55) -> FH12-24S-0.5SH(55)
Changed lines of the file:
@@
 L Connector_Generic:Conn_01x24 J2
 U 1 1 5B7B0E50
-P 10850 2050
-F 0 "J2" H 10769 625 50  0000 C CNN
-F 1 "FH12A-24S-0.5SH(55)" H 10769 716 50  0000 C CNN
-F 2 "exa_tim:Hirose_FH12-24S-0.5SH_1x24-1MP_P0.50mm_Horizontal" H 10850 2050 50  0001 C CNN
-F 3 "https://www.mouser.de/datasheet/2/185/FH12_catalog-939276.pdf" H 10850 2050 50  0001 C CNN
-	1    10850 2050
-	1    0    0    1
+P 10850 1950
+F 0 "J2" H 10769 525 50  0000 C CNN
+F 1 "FH12-24S-0.5SH(55)" H 10769 616 50  0000 C CNN
+F 2 "exa_tim:Hirose_FH12-24S-0.5SH_1x24-1MP_P0.50mm_Horizontal" H 10850 1950 50  0001 C CNN
+F 3 "https://www.mouser.de/datasheet/2/185/FH12_catalog-939276.pdf" H 10850 1950 50  0001 C CNN
+	1    10850 1950
+	1    0    0    -1
 $EndComp
 Text Label 10250 950  0    50   ~ 0

Commit message: Change battery to CR2032 for better height profile
Parts:
- BT1: value NL5077-LF -> 3034TR; footprint exa_tim:NL5077-LF -> exa_tim:BatteryHolder_Keystone_3034_1x20mm; Notice CR2450 or CR2477 -> CR2032
Changed lines of the file:
@@
 P 900 4150
 F 0 "BT1" H 1018 4246 50  0000 L CNN
-F 1 "NL5077-LF" H 1018 4155 50  0000 L CNN
-F 2 "exa_tim:NL5077-LF" V 900 4210 50  0001 C CNN
-F 3 "~" V 900 4210 50  0001 C CNN
-F 4 "CR2450 or CR2477" H 900 4150 50  0001 C CNN "Notice"
+F 1 "3034TR" H 1018 4155 50  0000 L CNN
+F 2 "exa_tim:BatteryHolder_Keystone_3034_1x20mm" V 900 4210 50  0001 C CNN
+F 3 "http://www.keyelco.com/product-pdf.cfm?p=798" V 900 4210 50  0001 C CNN
+F 4 "CR2032" H 900 4150 50  0001 C CNN "Notice"
 	1    900  4150
 	1    0    0    -1

Commit message: Use different buttons to get thinner design
I used other buttons and relocated the buttons and the
SWD connector to the bottom of the PCB to get a much
thinner design. PCB will use a 1mm board.
Parts:
- J1: value Conn_ARM_JTAG_SWD_10 -> 20021121-00010C4LF; footprint Connector_PinHeader_1.27mm:PinHeader_2x05_P1.27mm_Vertical_SMD -> exa_tim:PinHeader_2x05_P1.27mm_Vertical_SMD
- SW1, SW2, SW3, SW4: value SKHLLFA010 -> SKRTLBE010; footprint exa_tim:SKHLLFA010 -> exa_tim:SKRTLBE010
Changed lines of the file:
@@
 P 2350 6450
 F 0 "J1" H 1910 6496 50  0000 R CNN
-F 1 "Conn_ARM_JTAG_SWD_10" H 1910 6405 50  0000 R CNN
-F 2 "Connector_PinHeader_1.27mm:PinHeader_2x05_P1.27mm_Vertical_SMD" H 2400 5900 50  0001 L TNN
+F 1 "20021121-00010C4LF" H 1910 6405 50  0000 R CNN
+F 2 "exa_tim:PinHeader_2x05_P1.27mm_Vertical_SMD" H 2400 5900 50  0001 L TNN
 F 3 "http://infocenter.arm.com/help/topic/com.arm.doc.faqs/attached/13634/cortex_debug_connectors.pdf" V 2000 5200 50  0001 C CNN
 	1    2350 6450
@@
 P 5650 6050
 F 0 "SW4" H 5650 6285 50  0000 C CNN
-F 1 "SKHLLFA010" H 5650 6194 50  0000 C CNN
-F 2 "exa_tim:SKHLLFA010" H 5650 6050 50  0001 C CNN
-F 3 "https://www.mouser.de/datasheet/2/15/SKHL-1370655.pdf" H 5650 6050 50  0001 C CNN
+F 1 "SKRTLBE010" H 5650 6194 50  0000 C CNN
+F 2 "exa_tim:SKRTLBE010" H 5650 6050 50  0001 C CNN
+F 3 "https://www.alps.com/prod/info/E/PDF/Tact/SurfaceMount/SKRT/SKRTLBE010.pdf" H 5650 6050 50  0001 C CNN
 	1    5650 6050
 	1    0    0    -1
@@
 P 5650 4450
 F 0 "SW1" H 5650 4685 50  0000 C CNN
-F 1 "SKHLLFA010" H 5650 4594 50  0000 C CNN
-F 2 "exa_tim:SKHLLFA010" H 5650 4450 50  0001 C CNN
-F 3 "https://www.mouser.de/datasheet/2/15/SKHL-1370655.pdf" H 5650 4450 50  0001 C CNN
+F 1 "SKRTLBE010" H 5650 4594 50  0000 C CNN
+F 2 "exa_tim:SKRTLBE010" H 5650 4450 50  0001 C CNN
+F 3 "https://www.alps.com/prod/info/E/PDF/Tact/SurfaceMount/SKRT/SKRTLBE010.pdf" H 5650 4450 50  0001 C CNN
 	1    5650 4450
 	1    0    0    -1
@@
 P 5650 5550
 F 0 "SW3" H 5650 5785 50  0000 C CNN
-F 1 "SKHLLFA010" H 5650 5694 50  0000 C CNN
-F 2 "exa_tim:SKHLLFA010" H 5650 5550 50  0001 C CNN
-F 3 "https://www.mouser.de/datasheet/2/15/SKHL-1370655.pdf" H 5650 5550 50  0001 C CNN
+F 1 "SKRTLBE010" H 5650 5694 50  0000 C CNN
+F 2 "exa_tim:SKRTLBE010" H 5650 5550 50  0001 C CNN
+F 3 "https://www.alps.com/prod/info/E/PDF/Tact/SurfaceMount/SKRT/SKRTLBE010.pdf" H 5650 5550 50  0001 C CNN
 	1    5650 5550
 	1    0    0    -1
@@
 P 5650 5000
 F 0 "SW2" H 5650 5235 50  0000 C CNN
-F 1 "SKHLLFA010" H 5650 5144 50  0000 C CNN
-F 2 "exa_tim:SKHLLFA010" H 5650 5000 50  0001 C CNN
-F 3 "https://www.mouser.de/datasheet/2/15/SKHL-1370655.pdf" H 5650 5000 50  0001 C CNN
+F 1 "SKRTLBE010" H 5650 5144 50  0000 C CNN
+F 2 "exa_tim:SKRTLBE010" H 5650 5000 50  0001 C CNN
+F 3 "https://www.alps.com/prod/info/E/PDF/Tact/SurfaceMount/SKRT/SKRTLBE010.pdf" H 5650 5000 50  0001 C CNN
 	1    5650 5000
 	1    0    0    -1

Commit message: Revert PCB cutout and change button layout
Buttons are not top facing for easier assembly.
First inner layer is now power lane.
Removed useless LED, since we have no way to illuminate
the epaper display.
Parts:
- removed D1: LTST-C194KSKT, LED_SMD:LED_0603_1608Metric, symbol Device:LED_ALT
- removed R2: 1k, Resistor_SMD:R_0603_1608Metric, symbol Device:R
- SW1, SW2, SW3, SW4: value SKRTLBE010 -> TL3305CF260QG; footprint exa_tim:SKRTLBE010 -> exa_tim:TL3305
- Y1: footprint Crystal:Crystal_SMD_TXC_9HT11-2Pin_2.0x1.2mm -> exa_tim:Crystal_SMD_TXC_9HT11-2Pin_2.0x1.2mm_HandSoldering
- renumbered D2 to D1, D3 to D2, D4 to D3, D5 to D4, D6 to D5, D7 to D6, D8 to D7, R3 to R2, R4 to R3, R5 to R4, R6 to R5, R7 to R6, R8 to R7
Connections:
- net labels removed: LED
- wire segments 193 -> 189
Changed lines of the file:
@@
 F 0 "Y1" V 1900 2450 50  0000 C CNN
 F 1 "9HT11-32.768KDZF-T" V 1450 2450 50  0000 C CNN
-F 2 "Crystal:Crystal_SMD_TXC_9HT11-2Pin_2.0x1.2mm" H 1700 2450 50  0001 C CNN
+F 2 "exa_tim:Crystal_SMD_TXC_9HT11-2Pin_2.0x1.2mm_HandSoldering" H 1700 2450 50  0001 C CNN
 F 3 "http://www.txccrystal.com/images/pdf/9ht11.pdf" H 1700 2450 50  0001 C CNN
 	1    1700 2450
@@
 Text Label 4050 2300 2    50   ~ 0
 SCK
-Text Label 4050 2400 2    50   ~ 0
+Text Label 4050 2600 2    50   ~ 0
 CS
 Text Label 4050 2500 2    50   ~ 0
 MOSI
-Text Label 4050 2600 2    50   ~ 0
+Text Label 4050 2400 2    50   ~ 0
 BUSY
-Text Label 4050 2700 2    50   ~ 0
-LED
 Wire Wire Line
 	4050 1800 3400 1800
@@
 	9400 2450 9400 2200
 $Comp
-L Device:D_Schottky_ALT D6
+L Device:D_Schottky_ALT D5
 U 1 1 5B84CDBF
 P 10300 4000
-F 0 "D6" H 10300 4216 50  0000 C CNN
+F 0 "D5" H 10300 4216 50  0000 C CNN
 F 1 "MBR0530" H 10300 4125 50  0000 C CNN
 F 2 "Diode_SMD:D_SOD-123" H 10300 4000 50  0001 C CNN
@@
 $EndComp
 $Comp
-L Device:D_Schottky_ALT D7
+L Device:D_Schottky_ALT D6
 U 1 1 5B85311F
 P 10300 4550
-F 0 "D7" H 10300 4766 50  0000 C CNN
+F 0 "D6" H 10300 4766 50  0000 C CNN
 F 1 "MBR0530" H 10300 4675 50  0000 C CNN
 F 2 "Diode_SMD:D_SOD-123" H 10300 4550 50  0001 C CNN
@@
 PREVGH
 $Comp
-L Device:D_Schottky_ALT D8
+L Device:D_Schottky_ALT D7
 U 1 1 5B86AB68
 P 10300 4850
-F 0 "D8" H 10300 5066 50  0000 C CNN
+F 0 "D7" H 10300 5066 50  0000 C CNN
 F 1 "MBR0530" H 10300 4975 50  0000 C CNN
 F 2 "Diode_SMD:D_SOD-123" H 10300 4850 50  0001 C CNN
@@
 GDR
 $Comp
-L Device:R R7
+L Device:R R6
 U 1 1 5B8A6DE8
 P 9150 5850
-F 0 "R7" H 9220 5896 50  0000 L CNN
+F 0 "R6" H 9220 5896 50  0000 L CNN
 F 1 "1M" H 9220 5805 50  0000 L CNN
 F 2 "Resistor_SMD:R_0603_1608Metric" V 9080 5850 50  0001 C CNN
@@
 $EndComp
 $Comp
-L Device:R R8
+L Device:R R7
 U 1 1 5B8AB1E0
 P 9550 5850
-F 0 "R8" H 9620 5896 50  0000 L CNN
+F 0 "R7" H 9620 5896 50  0000 L CNN
 F 1 "3" H 9620 5805 50  0000 L CNN
 F 2 "Resistor_SMD:R_0603_1608Metric" V 9480 5850 50  0001 C CNN
@@
 P 5650 6050
 F 0 "SW4" H 5650 6285 50  0000 C CNN
-F 1 "SKRTLBE010" H 5650 6194 50  0000 C CNN
-F 2 "exa_tim:SKRTLBE010" H 5650 6050 50  0001 C CNN
-F 3 "https://www.alps.com/prod/info/E/PDF/Tact/SurfaceMount/SKRT/SKRTLBE010.pdf" H 5650 6050 50  0001 C CNN
+F 1 "TL3305CF260QG" H 5650 6194 50  0000 C CNN
+F 2 "exa_tim:TL3305" H 5650 6050 50  0001 C CNN
+F 3 "https://www.mouser.de/datasheet/2/140/TL3305-844809.pdf" H 5650 6050 50  0001 C CNN
 	1    5650 6050
 	1    0    0    -1
@@
 P 5650 4450
 F 0 "SW1" H 5650 4685 50  0000 C CNN
-F 1 "SKRTLBE010" H 5650 4594 50  0000 C CNN
-F 2 "exa_tim:SKRTLBE010" H 5650 4450 50  0001 C CNN
-F 3 "https://www.alps.com/prod/info/E/PDF/Tact/SurfaceMount/SKRT/SKRTLBE010.pdf" H 5650 4450 50  0001 C CNN
+F 1 "TL3305CF260QG" H 5650 4594 50  0000 C CNN
+F 2 "exa_tim:TL3305" H 5650 4450 50  0001 C CNN
+F 3 "https://www.mouser.de/datasheet/2/140/TL3305-844809.pdf" H 5650 4450 50  0001 C CNN
 	1    5650 4450
 	1    0    0    -1
@@
 P 5650 5550
 F 0 "SW3" H 5650 5785 50  0000 C CNN
-F 1 "SKRTLBE010" H 5650 5694 50  0000 C CNN
-F 2 "exa_tim:SKRTLBE010" H 5650 5550 50  0001 C CNN
-F 3 "https://www.alps.com/prod/info/E/PDF/Tact/SurfaceMount/SKRT/SKRTLBE010.pdf" H 5650 5550 50  0001 C CNN
+F 1 "TL3305CF260QG" H 5650 5694 50  0000 C CNN
+F 2 "exa_tim:TL3305" H 5650 5550 50  0001 C CNN
+F 3 "https://www.mouser.de/datasheet/2/140/TL3305-844809.pdf" H 5650 5550 50  0001 C CNN
 	1    5650 5550
 	1    0    0    -1
@@
 P 5650 5000
 F 0 "SW2" H 5650 5235 50  0000 C CNN
-F 1 "SKRTLBE010" H 5650 5144 50  0000 C CNN
-F 2 "exa_tim:SKRTLBE010" H 5650 5000 50  0001 C CNN
-F 3 "https://www.alps.com/prod/info/E/PDF/Tact/SurfaceMount/SKRT/SKRTLBE010.pdf" H 5650 5000 50  0001 C CNN
+F 1 "TL3305CF260QG" H 5650 5144 50  0000 C CNN
+F 2 "exa_tim:TL3305" H 5650 5000 50  0001 C CNN
+F 3 "https://www.mouser.de/datasheet/2/140/TL3305-844809.pdf" H 5650 5000 50  0001 C CNN
 	1    5650 5000
 	1    0    0    -1
@@
 NoConn ~ 5250 2200
 $Comp
-L Device:R R5
+L Device:R R4
 U 1 1 5B819EC8
 P 7050 3000
-F 0 "R5" V 6843 3000 50  0000 C CNN
+F 0 "R4" V 6843 3000 50  0000 C CNN
 F 1 "220" V 6934 3000 50  0000 C CNN
 F 2 "Resistor_SMD:R_0603_1608Metric" V 6980 3000 50  0001 C CNN
@@
 $EndComp
 $Comp
-L Device:R R6
+L Device:R R5
 U 1 1 5B81AB2F
 P 7050 3350
-F 0 "R6" V 6843 3350 50  0000 C CNN
+F 0 "R5" V 6843 3350 50  0000 C CNN
 F 1 "220" V 6934 3350 50  0000 C CNN
 F 2 "Resistor_SMD:R_0603_1608Metric" V 6980 3350 50  0001 C CNN
@@
 $EndComp
 $Comp
-L Device:R R4
+L Device:R R3
 U 1 1 5B8F6DF3
 P 5300 2950
-F 0 "R4" H 5370 2996 50  0000 L CNN
+F 0 "R3" H 5370 2996 50  0000 L CNN
 F 1 "1M" H 5370 2905 50  0000 L CNN
 F 2 "Resistor_SMD:R_0603_1608Metric" V 5230 2950 50  0001 C CNN
@@
 Wire Wire Line
 	4050 2600 3400 2600
-Wire Wire Line
-	3400 2700 4050 2700
 $Comp
 L Device:C C7
@@
 	2500 1400 2700 1400
 $Comp
-L Device:D_Schottky_ALT D5
+L Device:D_Schottky_ALT D4
 U 1 1 5BCC1FAE
 P 6750 6050
-F 0 "D5" H 6750 6266 50  0000 C CNN
+F 0 "D4" H 6750 6266 50  0000 C CNN
 F 1 "MBR0530" H 6750 6175 50  0000 C CNN
 F 2 "Diode_SMD:D_SOD-123" H 6750 6050 50  0001 C CNN
@@
 $EndComp
 $Comp
-L Device:D_Schottky_ALT D2
+L Device:D_Schottky_ALT D1
 U 1 1 5BCCD658
 P 6750 4450
-F 0 "D2" H 6750 4666 50  0000 C CNN
+F 0 "D1" H 6750 4666 50  0000 C CNN
 F 1 "MBR0530" H 6750 4575 50  0000 C CNN
 F 2 "Diode_SMD:D_SOD-123" H 6750 4450 50  0001 C CNN
@@
 $EndComp
 $Comp
-L Device:D_Schottky_ALT D4
+L Device:D_Schottky_ALT D3
 U 1 1 5BCE28FC
 P 6750 5550
-F 0 "D4" H 6750 5766 50  0000 C CNN
+F 0 "D3" H 6750 5766 50  0000 C CNN
 F 1 "MBR0530" H 6750 5675 50  0000 C CNN
 F 2 "Diode_SMD:D_SOD-123" H 6750 5550 50  0001 C CNN
@@
 $EndComp
 $Comp
-L Device:D_Schottky_ALT D3
+L Device:D_Schottky_ALT D2
 U 1 1 5BCED23B
 P 6750 5000
-F 0 "D3" H 6750 5216 50  0000 C CNN
+F 0 "D2" H 6750 5216 50  0000 C CNN
 F 1 "MBR0530" H 6750 5125 50  0000 C CNN
 F 2 "Diode_SMD:D_SOD-123" H 6750 5000 50  0001 C CNN
@@
 Connection ~ 4850 5550
 $Comp
-L Device:LED_ALT D1
-U 1 1 5BE0EA43
-P 2750 4600
-F 0 "D1" H 2742 4345 50  0000 C CNN
-F 1 "LTST-C194KSKT" H 2742 4436 50  0000 C CNN
-F 2 "LED_SMD:LED_0603_1608Metric" H 2750 4600 50  0001 C CNN
-F 3 "~" H 2750 4600 50  0001 C CNN
-	1    2750 4600
-	-1   0    0    1
-$EndComp
-Text Label 1900 4600 0    50   ~ 0
-LED
-$Comp
-L Device:R R2
-U 1 1 5BE0FB49
-P 2300 4600
-F 0 "R2" V 2507 4600 50  0000 C CNN
-F 1 "1k" V 2416 4600 50  0000 C CNN
-F 2 "Resistor_SMD:R_0603_1608Metric" V 2230 4600 50  0001 C CNN
-F 3 "~" H 2300 4600 50  0001 C CNN
-	1    2300 4600
-	0    -1   -1   0
-$EndComp
-Wire Wire Line
-	1900 4600 2150 4600
-Wire Wire Line
-	2450 4600 2600 4600
-$Comp
-L power:GND #PWR09
-U 1 1 5BE34009
-P 3100 4600
-F 0 "#PWR09" H 3100 4350 50  0001 C CNN
-F 1 "GND" H 3105 4427 50  0000 C CNN
-F 2 "" H 3100 4600 50  0001 C CNN
-F 3 "" H 3100 4600 50  0001 C CNN
-	1    3100 4600
-	0    -1   -1   0
-$EndComp
-Wire Wire Line
-	3100 4600 2900 4600
-$Comp
 L Device:Speaker LS1
 U 1 1 5BEA6795
@@
 $EndComp
 $Comp
-L Device:R R3
+L Device:R R2
 U 1 1 5BEA68C0
 P 2450 5150
-F 0 "R3" V 2243 5150 50  0000 C CNN
+F 0 "R2" V 2243 5150 50  0000 C CNN
 F 1 "220" V 2334 5150 50  0000 C CNN
 F 2 "Resistor_SMD:R_0603_1608Metric" V 2380 5150 50  0001 C CNN
@@
 	0    -1   -1   0
 $EndComp
+$Comp
+L power:GND #PWR09
+U 1 1 5B8876BC
+P 3400 2700
+F 0 "#PWR09" H 3400 2450 50  0001 C CNN
+F 1 "GND" V 3405 2572 50  0000 R CNN
+F 2 "" H 3400 2700 50  0001 C CNN
+F 3 "" H 3400 2700 50  0001 C CNN
+	1    3400 2700
+	0    -1   -1   0
+$EndComp

Commit message: Chang Cortex Debug header to right angle TH
Parts:
- J1: value 20021121-00010C4LF -> 20021112-00010T4LF; footprint exa_tim:PinHeader_2x05_P1.27mm_Vertical_SMD -> Connector_PinHeader_1.27mm:PinHeader_2x06_P1.27mm_Horizontal
Changed lines of the file:
@@
 P 2350 6450
 F 0 "J1" H 1910 6496 50  0000 R CNN
-F 1 "20021121-00010C4LF" H 1910 6405 50  0000 R CNN
-F 2 "exa_tim:PinHeader_2x05_P1.27mm_Vertical_SMD" H 2400 5900 50  0001 L TNN
+F 1 "20021112-00010T4LF" H 1910 6405 50  0000 R CNN
+F 2 "Connector_PinHeader_1.27mm:PinHeader_2x06_P1.27mm_Horizontal" H 2400 5900 50  0001 L TNN
 F 3 "http://infocenter.arm.com/help/topic/com.arm.doc.faqs/attached/13634/cortex_debug_connectors.pdf" V 2000 5200 50  0001 C CNN
 	1    2350 6450
