File: PCB/exa_tim.sch (KiCad schematic (older format))
At the start: 52 parts, among them J1 20021112-00010T4LF, J2 FH12-24S-0.5SH(55), Q1 SI2333DS-T1-E3, Q2 DMN3067LW-7, SW1 TL3305CF260QG, SW2 TL3305CF260QG, SW3 TL3305CF260QG, SW4 TL3305CF260QG, U1 STM32L071KZUx, U2 CAM-M8C-0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

Commit message: Change crystal caps from 21 to 20pF
Parts:
- C2, C3: value 21pF -> 20pF
Changed lines of the file:
@@
 P 1400 2350
 F 0 "C2" V 1700 2200 50  0000 L CNN
-F 1 "21pF" V 1800 2200 50  0000 L CNN
+F 1 "20pF" V 1800 2200 50  0000 L CNN
 F 2 "Capacitor_SMD:C_0603_1608Metric" H 1400 2350 50  0001 C CNN
 F 3 "~" H 1400 2350 50  0001 C CNN
@@
 P 1400 2550
 F 0 "C3" V 1500 2600 50  0000 L CNN
-F 1 "21pF" V 1600 2600 50  0000 L CNN
+F 1 "20pF" V 1600 2600 50  0000 L CNN
 F 2 "Capacitor_SMD:C_0603_1608Metric" H 1400 2550 50  0001 C CNN
 F 3 "~" H 1400 2550 50  0001 C CNN
