File: pcb/exa_tim.sch (KiCad schematic (older format))
At the start: 52 parts, among them J1 20021112-00010T4LF, J2 FH12-24S-0.5SH(55), Q1 SI2333DS-T1-E3, Q2 DMN3067LW-7, SW1 TL3305CF260QG, SW2 TL3305CF260QG, SW3 TL3305CF260QG, SW4 TL3305CF260QG, U1 STM32L071KZUx, U2 CAM-M8C-0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

Commit message: Changed 2x06 header to 2x05 header
I choosed the wrong header for the Cortex Debug header.
This is the correct header. The old header is working fine
but two holes are not used.
Parts:
- J1: footprint Connector_PinHeader_1.27mm:PinHeader_2x06_P1.27mm_Horizontal -> Connector_PinHeader_1.27mm:PinHeader_2x05_P1.27mm_Horizontal
Changed lines of the file:
@@
 F 0 "J1" H 1910 6496 50  0000 R CNN
 F 1 "20021112-00010T4LF" H 1910 6405 50  0000 R CNN
-F 2 "Connector_PinHeader_1.27mm:PinHeader_2x06_P1.27mm_Horizontal" H 2400 5900 50  0001 L TNN
+F 2 "Connector_PinHeader_1.27mm:PinHeader_2x05_P1.27mm_Horizontal" H 2400 5900 50  0001 L TNN
 F 3 "http://infocenter.arm.com/help/topic/com.arm.doc.faqs/attached/13634/cortex_debug_connectors.pdf" V 2000 5200 50  0001 C CNN
 	1    2350 6450

Commit message: Fix p-channel MOSFET and new routing
Fixed the p-channel MOSFET drain/source problem (was reversed).
New placement for the SWO header (2x05) for easier placement.
Re-routed signals, so that ground and power lane are signal trace
free.
Connections:
- wire segments 189 -> 188
Changed lines of the file:
@@
 L Device:R R3
 U 1 1 5B8F6DF3
-P 5300 2950
-F 0 "R3" H 5370 2996 50  0000 L CNN
-F 1 "1M" H 5370 2905 50  0000 L CNN
-F 2 "Resistor_SMD:R_0603_1608Metric" V 5230 2950 50  0001 C CNN
-F 3 "~" H 5300 2950 50  0001 C CNN
-	1    5300 2950
+P 5300 3400
+F 0 "R3" H 5370 3446 50  0000 L CNN
+F 1 "1M" H 5370 3355 50  0000 L CNN
+F 2 "Resistor_SMD:R_0603_1608Metric" V 5230 3400 50  0001 C CNN
+F 3 "~" H 5300 3400 50  0001 C CNN
+	1    5300 3400
 	1    0    0    -1
 $EndComp
@@
 Wire Wire Line
 	4900 3250 5300 3250
-Wire Wire Line
-	5300 3250 5300 3100
 Connection ~ 5300 3250
 Wire Wire Line
 	5300 3250 5500 3250
-Wire Wire Line
-	5800 3050 5800 2700
-Wire Wire Line
-	5800 2700 5300 2700
-Wire Wire Line
-	5300 2700 5300 2800
-Text Label 5800 3650 0    50   ~ 0
+Text Label 5800 2850 0    50   ~ 0
 GNSS_VDD
-Text GLabel 5800 2700 2    50   Input ~ 0
+Text GLabel 5800 3650 2    50   Input ~ 0
 3V
 Text Label 7750 1300 0    50   ~ 0
@@
 	0    -1   -1   0
 $EndComp
+Wire Wire Line
+	5800 3650 5300 3650
+Wire Wire Line
+	5300 3650 5300 3550
+Wire Wire Line
+	5800 3050 5800 2850
 $EndSCHEMATC

Commit message: Add new font, add alarm, removed alarm series resistor
The series resistor was not needed, since the alarm would be too
tiny. I also added basic "beep" functionality.

Also added a new font face size 96.
Parts:
- removed R2: 220, Resistor_SMD:R_0603_1608Metric, symbol Device:R
- renumbered R3 to R2, R4 to R3, R5 to R4, R6 to R5, R7 to R6
Connections:
- wire segments 188 -> 187
Changed lines of the file:
@@
 GDR
 $Comp
-L Device:R R6
+L Device:R R5
 U 1 1 5B8A6DE8
 P 9150 5850
-F 0 "R6" H 9220 5896 50  0000 L CNN
+F 0 "R5" H 9220 5896 50  0000 L CNN
 F 1 "1M" H 9220 5805 50  0000 L CNN
 F 2 "Resistor_SMD:R_0603_1608Metric" V 9080 5850 50  0001 C CNN
@@
 $EndComp
 $Comp
-L Device:R R7
+L Device:R R6
 U 1 1 5B8AB1E0
 P 9550 5850
-F 0 "R7" H 9620 5896 50  0000 L CNN
+F 0 "R6" H 9620 5896 50  0000 L CNN
 F 1 "3" H 9620 5805 50  0000 L CNN
 F 2 "Resistor_SMD:R_0603_1608Metric" V 9480 5850 50  0001 C CNN
@@
 NoConn ~ 5250 2200
 $Comp
-L Device:R R4
+L Device:R R3
 U 1 1 5B819EC8
 P 7050 3000
-F 0 "R4" V 6843 3000 50  0000 C CNN
+F 0 "R3" V 6843 3000 50  0000 C CNN
 F 1 "220" V 6934 3000 50  0000 C CNN
 F 2 "Resistor_SMD:R_0603_1608Metric" V 6980 3000 50  0001 C CNN
@@
 $EndComp
 $Comp
-L Device:R R5
+L Device:R R4
 U 1 1 5B81AB2F
 P 7050 3350
-F 0 "R5" V 6843 3350 50  0000 C CNN
+F 0 "R4" V 6843 3350 50  0000 C CNN
 F 1 "220" V 6934 3350 50  0000 C CNN
 F 2 "Resistor_SMD:R_0603_1608Metric" V 6980 3350 50  0001 C CNN
@@
 $EndComp
 $Comp
-L Device:R R3
+L Device:R R2
 U 1 1 5B8F6DF3
 P 5300 3400
-F 0 "R3" H 5370 3446 50  0000 L CNN
+F 0 "R2" H 5370 3446 50  0000 L CNN
 F 1 "1M" H 5370 3355 50  0000 L CNN
 F 2 "Resistor_SMD:R_0603_1608Metric" V 5230 3400 50  0001 C CNN
@@
 $EndComp
 $Comp
-L Device:R R2
-U 1 1 5BEA68C0
-P 2450 5150
-F 0 "R2" V 2243 5150 50  0000 C CNN
-F 1 "220" V 2334 5150 50  0000 C CNN
-F 2 "Resistor_SMD:R_0603_1608Metric" V 2380 5150 50  0001 C CNN
-F 3 "~" H 2450 5150 50  0001 C CNN
-	1    2450 5150
-	0    1    1    0
-$EndComp
-$Comp
 L power:GND #PWR05
 U 1 1 5BEA69F0
@@
 ALARM
 Wire Wire Line
-	1950 5150 2300 5150
-Wire Wire Line
-	2600 5150 2800 5150
-Wire Wire Line
 	2800 5250 1950 5250
 Wire Wire Line
@@
 Wire Wire Line
 	5800 3050 5800 2850
+Wire Wire Line
+	1950 5150 2800 5150
 $EndSCHEMATC

Commit message: Chang GNSS MOSFET to enh. N-Channel
Changed the MOSFET so that we don't need a pullup,
which might draw some precious power we don't want to
waste.

Also simplifies the BOM.
Parts:
- removed Q1: SI2333DS-T1-E3, Package_TO_SOT_SMD:SOT-23, symbol Device:Q_PMOS_GSD
- added Q1: DMN3067LW-7, Package_TO_SOT_SMD:SOT-323_SC-70, symbol Device:Q_NMOS_GSD
Connections:
- net labels added: GNSS_GND
- net labels removed: GNSS_VDD
Changed lines of the file:
@@
 NoConn ~ 7450 2200
 NoConn ~ 7450 1800
-$Comp
-L power:GND #PWR013
-U 1 1 5B7F342C
-P 7450 2400
-F 0 "#PWR013" H 7450 2150 50  0001 C CNN
-F 1 "GND" V 7455 2272 50  0000 R CNN
-F 2 "" H 7450 2400 50  0001 C CNN
-F 3 "" H 7450 2400 50  0001 C CNN
-	1    7450 2400
-	0    -1   -1   0
-$EndComp
 Text Label 7750 1700 2    50   ~ 0
 TX_GNSS
@@
 GNSS_EN
 $Comp
-L Device:Q_PMOS_GSD Q1
-U 1 1 5B8EE47B
-P 5700 3250
-F 0 "Q1" H 5905 3296 50  0000 L CNN
-F 1 "SI2333DS-T1-E3" H 5905 3205 50  0000 L CNN
-F 2 "Package_TO_SOT_SMD:SOT-23" H 5900 3350 50  0001 C CNN
-F 3 "https://www.vishay.com/docs/72023/72023.pdf" H 5700 3250 50  0001 C CNN
-	1    5700 3250
-	1    0    0    -1
-$EndComp
-$Comp
 L Device:R R2
 U 1 1 5B8F6DF3
@@
 $EndComp
 Wire Wire Line
-	5800 3450 5800 3650
+	5800 3450 5800 3550
 Text Label 4900 3250 0    50   ~ 0
 GNSS_EN
@@
 Wire Wire Line
 	5300 3250 5500 3250
-Text Label 5800 2850 0    50   ~ 0
-GNSS_VDD
-Text GLabel 5800 3650 2    50   Input ~ 0
+Text GLabel 7750 1300 2    50   Input ~ 0
 3V
-Text Label 7750 1300 0    50   ~ 0
-GNSS_VDD
 $Comp
 L MCU_ST_STM32L0:STM32L071KZUx U1
@@
 $EndComp
 Wire Wire Line
-	5800 3650 5300 3650
-Wire Wire Line
-	5300 3650 5300 3550
-Wire Wire Line
 	5800 3050 5800 2850
 Wire Wire Line
 	1950 5150 2800 5150
+$Comp
+L Device:Q_NMOS_GSD Q1
+U 1 1 5B9F4C7F
+P 5700 3250
+F 0 "Q1" H 5906 3296 50  0000 L CNN
+F 1 "DMN3067LW-7" H 5906 3205 50  0000 L CNN
+F 2 "Package_TO_SOT_SMD:SOT-323_SC-70" H 5900 3350 50  0001 C CNN
+F 3 "https://www.mouser.de/datasheet/2/115/DMN3067LW-335715.pdf" H 5700 3250 50  0001 C CNN
+	1    5700 3250
+	1    0    0    -1
+$EndComp
+Text Label 7450 2400 0    50   ~ 0
+GNSS_GND
+Text Label 5800 2850 0    50   ~ 0
+GNSS_GND
+$Comp
+L power:GND #PWR013
+U 1 1 5BA6FCEF
+P 5800 3650
+F 0 "#PWR013" H 5800 3400 50  0001 C CNN
+F 1 "GND" H 5805 3477 50  0000 C CNN
+F 2 "" H 5800 3650 50  0001 C CNN
+F 3 "" H 5800 3650 50  0001 C CNN
+	1    5800 3650
+	1    0    0    -1
+$EndComp
+Wire Wire Line
+	5300 3550 5800 3550
+Connection ~ 5800 3550
+Wire Wire Line
+	5800 3550 5800 3650
 $EndSCHEMATC

Commit message: First pass to re-arange parts to move connector
Changed lines of the file:
@@
 Text Label 1900 3200 0    50   ~ 0
 BTN4
-Text Label 1900 2900 0    50   ~ 0
+Text Label 1900 3000 0    50   ~ 0
 BTN1
 Text Label 1900 3100 0    50   ~ 0
@@
 NoConn ~ 10650 1350
 NoConn ~ 10650 1450
-Text Label 1900 3000 0    50   ~ 0
+Text Label 1900 2900 0    50   ~ 0
 BTN2
 Wire Wire Line

Commit message: Switched backt to high side p-channel MOSFET
I don't want to risk communication errros of UART
because of the otherwise not common ground levels.
Parts:
- C2, C3: value 20pF -> 4pF
- Q1: value DMN3067LW-7 -> SI2333DS-T1-E3; footprint Package_TO_SOT_SMD:SOT-323_SC-70 -> Package_TO_SOT_SMD:SOT-23; symbol Device:Q_NMOS_GSD -> Device:Q_PMOS_GSD
- Y1: value 9HT11-32.768KDZF-T -> 9HT11-32.768KDZB-T
Connections:
- net labels added: VDD_GNSS
- net labels removed: GNSS_GND
Changed lines of the file:
@@
 P 1700 2450
 F 0 "Y1" V 1900 2450 50  0000 C CNN
-F 1 "9HT11-32.768KDZF-T" V 1450 2450 50  0000 C CNN
+F 1 "9HT11-32.768KDZB-T" V 1450 2450 50  0000 C CNN
 F 2 "exa_tim:Crystal_SMD_TXC_9HT11-2Pin_2.0x1.2mm_HandSoldering" H 1700 2450 50  0001 C CNN
 F 3 "http://www.txccrystal.com/images/pdf/9ht11.pdf" H 1700 2450 50  0001 C CNN
@@
 P 1400 2350
 F 0 "C2" V 1700 2200 50  0000 L CNN
-F 1 "20pF" V 1800 2200 50  0000 L CNN
+F 1 "4pF" V 1800 2200 50  0000 L CNN
 F 2 "Capacitor_SMD:C_0603_1608Metric" H 1400 2350 50  0001 C CNN
 F 3 "~" H 1400 2350 50  0001 C CNN
@@
 P 1400 2550
 F 0 "C3" V 1500 2600 50  0000 L CNN
-F 1 "20pF" V 1600 2600 50  0000 L CNN
+F 1 "4pF" V 1600 2600 50  0000 L CNN
 F 2 "Capacitor_SMD:C_0603_1608Metric" H 1400 2550 50  0001 C CNN
 F 3 "~" H 1400 2550 50  0001 C CNN
@@
 Wire Wire Line
 	5300 3250 5500 3250
-Text GLabel 7750 1300 2    50   Input ~ 0
+Text GLabel 5800 3650 2    50   Input ~ 0
 3V
 $Comp
@@
 $EndComp
 Wire Wire Line
-	5800 3050 5800 2850
-Wire Wire Line
 	1950 5150 2800 5150
 $Comp
-L Device:Q_NMOS_GSD Q1
+L Device:Q_PMOS_GSD Q1
 U 1 1 5B9F4C7F
 P 5700 3250
 F 0 "Q1" H 5906 3296 50  0000 L CNN
-F 1 "DMN3067LW-7" H 5906 3205 50  0000 L CNN
-F 2 "Package_TO_SOT_SMD:SOT-323_SC-70" H 5900 3350 50  0001 C CNN
-F 3 "https://www.mouser.de/datasheet/2/115/DMN3067LW-335715.pdf" H 5700 3250 50  0001 C CNN
+F 1 "SI2333DS-T1-E3" H 5906 3205 50  0000 L CNN
+F 2 "Package_TO_SOT_SMD:SOT-23" H 5900 3350 50  0001 C CNN
+F 3 "https://www.vishay.com/docs/72023/72023.pdf" H 5700 3250 50  0001 C CNN
 	1    5700 3250
-	1    0    0    -1
-$EndComp
-Text Label 7450 2400 0    50   ~ 0
-GNSS_GND
-Text Label 5800 2850 0    50   ~ 0
-GNSS_GND
-$Comp
-L power:GND #PWR013
-U 1 1 5BA6FCEF
-P 5800 3650
-F 0 "#PWR013" H 5800 3400 50  0001 C CNN
-F 1 "GND" H 5805 3477 50  0000 C CNN
-F 2 "" H 5800 3650 50  0001 C CNN
-F 3 "" H 5800 3650 50  0001 C CNN
-	1    5800 3650
 	1    0    0    -1
 $EndComp
@@
 Wire Wire Line
 	5800 3550 5800 3650
+$Comp
+L power:GND #PWR?
+U 1 1 5BA03A7E
+P 7450 2400
+F 0 "#PWR?" H 7450 2150 50  0001 C CNN
+F 1 "GND" H 7455 2227 50  0000 C CNN
+F 2 "" H 7450 2400 50  0001 C CNN
+F 3 "" H 7450 2400 50  0001 C CNN
+	1    7450 2400
+	0    -1   -1   0
+$EndComp
+Wire Wire Line
+	5800 3050 5800 2850
+Text Label 5800 2850 0    50   ~ 0
+VDD_GNSS
+Text Label 7750 1300 0    50   ~ 0
+VDD_GNSS
 $EndSCHEMATC

Commit message: Redesigned LSE layout and re-routed some traces
Also switched BTN3 and BTN4 pins for easier routing.
Parts:
- added R7: 0, Resistor_SMD:R_0603_1608Metric, symbol Device:R
Connections:
- net labels added: GNDD
Changed lines of the file:
@@
 Text Label 4050 3200 2    50   ~ 0
 SWCLK
-Text Label 1900 3200 0    50   ~ 0
+Text Label 1900 3100 0    50   ~ 0
 BTN4
 Text Label 1900 3000 0    50   ~ 0
 BTN1
-Text Label 1900 3100 0    50   ~ 0
+Text Label 1900 3200 0    50   ~ 0
 BTN3
 Wire Wire Line
@@
 	2800 5250 1950 5250
 Wire Wire Line
-	1900 3200 2200 3200
+	1900 3100 2200 3100
 Wire Wire Line
 	2200 3000 1900 3000
@@
 BTN2
 Wire Wire Line
-	1900 3100 2200 3100
+	1900 3200 2200 3200
 $Comp
 L Device:C C6
@@
 	5800 3550 5800 3650
 $Comp
-L power:GND #PWR?
+L power:GND #PWR024
 U 1 1 5BA03A7E
 P 7450 2400
-F 0 "#PWR?" H 7450 2150 50  0001 C CNN
+F 0 "#PWR024" H 7450 2150 50  0001 C CNN
 F 1 "GND" H 7455 2227 50  0000 C CNN
 F 2 "" H 7450 2400 50  0001 C CNN
@@
 Text Label 7750 1300 0    50   ~ 0
 VDD_GNSS
+$Comp
+L power:GNDD #PWR013
+U 1 1 5BA24559
+P 10650 6400
+F 0 "#PWR013" H 10650 6150 50  0001 C CNN
+F 1 "GNDD" H 10654 6245 50  0000 C CNN
+F 2 "" H 10650 6400 50  0001 C CNN
+F 3 "" H 10650 6400 50  0001 C CNN
+	1    10650 6400
+	0    1    1    0
+$EndComp
+$Comp
+L power:GND #PWR023
+U 1 1 5BA24653
+P 10950 6400
+F 0 "#PWR023" H 10950 6150 50  0001 C CNN
+F 1 "GND" H 10955 6227 50  0000 C CNN
+F 2 "" H 10950 6400 50  0001 C CNN
+F 3 "" H 10950 6400 50  0001 C CNN
+	1    10950 6400
+	0    -1   -1   0
+$EndComp
+$Comp
+L Device:R R7
+U 1 1 5BA6FAC8
+P 10800 6400
+F 0 "R7" V 10593 6400 50  0000 C CNN
+F 1 "0" V 10684 6400 50  0000 C CNN
+F 2 "Resistor_SMD:R_0603_1608Metric" V 10730 6400 50  0001 C CNN
+F 3 "~" H 10800 6400 50  0001 C CNN
+	1    10800 6400
+	0    1    1    0
+$EndComp
 $EndSCHEMATC

Commit message: Switched LSE crystall for achieving LOW drive capability
It seems my oscilloscope is interfering wit LSE
operation when measuring and having the LOW drive
capability on.

But the LSE seeem to work fine, since the RTC and LPTIM
seem to work fine under it.
Parts:
- Y1: value 9HT11-32.768KDZB-T -> ST2012SB32768B0HPWBB
Changed lines of the file:
@@
 P 1700 2450
 F 0 "Y1" V 1900 2450 50  0000 C CNN
-F 1 "9HT11-32.768KDZB-T" V 1450 2450 50  0000 C CNN
+F 1 "ST2012SB32768B0HPWBB" V 1450 2450 50  0000 C CNN
 F 2 "exa_tim:Crystal_SMD_TXC_9HT11-2Pin_2.0x1.2mm_HandSoldering" H 1700 2450 50  0001 C CNN
-F 3 "http://www.txccrystal.com/images/pdf/9ht11.pdf" H 1700 2450 50  0001 C CNN
+F 3 "https://www.mouser.de/datasheet/2/909/st2012sb_e-1316888.pdf" H 1700 2450 50  0001 C CNN
 	1    1700 2450
 	0    1    1    0
