File: pcb/exa_tim.sch (KiCad schematic (older format))
At the start: 52 parts, among them J1 20021112-00010T4LF, J2 FH12-24S-0.5SH(55), Q1 SI2333DS-T1-E3, Q2 DMN3067LW-7, SW1 TL3305CF260QG, SW2 TL3305CF260QG, SW3 TL3305CF260QG, SW4 TL3305CF260QG, U1 STM32L071KZUx, U2 CAM-M8C-0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

Commit message: Add third MOSFET to shutdown E-Paper driver
This will cut off the e-paper from any voltage source
and should result in an even lower power usage.
Parts:
- removed R7: 0, Resistor_SMD:R_0603_1608Metric, symbol Device:R
- added Q2: SI2333DS-T1-E3, Package_TO_SOT_SMD:SOT-23, symbol Device:Q_PMOS_GSD
- added R5: 1M, Resistor_SMD:R_0603_1608Metric, symbol Device:R
- renumbered Q2 to Q3, R5 to R6, R6 to R7
Connections:
- net labels added: DISP_EN, VDD_DISP
- net labels removed: GNDD
- wire segments 187 -> 192
Changed lines of the file:
@@
 Wire Wire Line
 	900  4350 900  4250
-Text GLabel 10400 2350 0    50   Input ~ 0
-3V
-Wire Wire Line
-	10400 2350 10500 2350
-Wire Wire Line
-	10500 2250 10500 2350
-Wire Wire Line
-	10500 2250 10650 2250
-Connection ~ 10500 2350
-Wire Wire Line
-	10500 2350 10650 2350
 $Comp
 L Device:C C18
@@
 $EndComp
 Wire Wire Line
-	10500 2250 10200 2250
-Wire Wire Line
 	10200 2250 10200 1950
 Wire Wire Line
 	10200 1950 9850 1950
-Connection ~ 10500 2250
 Wire Wire Line
 	10150 2200 9850 2200
@@
 $EndComp
 $Comp
-L Device:Q_NMOS_GSD Q2
+L Device:Q_NMOS_GSD Q3
 U 1 1 5B8A63F8
 P 9450 5350
-F 0 "Q2" H 9656 5396 50  0000 L CNN
+F 0 "Q3" H 9656 5396 50  0000 L CNN
 F 1 "DMN3067LW-7" H 9656 5305 50  0000 L CNN
 F 2 "Package_TO_SOT_SMD:SOT-323_SC-70" H 9650 5450 50  0001 C CNN
@@
 GDR
 $Comp
-L Device:R R5
+L Device:R R6
 U 1 1 5B8A6DE8
 P 9150 5850
-F 0 "R5" H 9220 5896 50  0000 L CNN
+F 0 "R6" H 9220 5896 50  0000 L CNN
 F 1 "1M" H 9220 5805 50  0000 L CNN
 F 2 "Resistor_SMD:R_0603_1608Metric" V 9080 5850 50  0001 C CNN
@@
 $EndComp
 $Comp
-L Device:R R6
+L Device:R R7
 U 1 1 5B8AB1E0
 P 9550 5850
-F 0 "R6" H 9620 5896 50  0000 L CNN
+F 0 "R7" H 9620 5896 50  0000 L CNN
 F 1 "3" H 9620 5805 50  0000 L CNN
 F 2 "Resistor_SMD:R_0603_1608Metric" V 9480 5850 50  0001 C CNN
@@
 Text Label 4050 2100 2    50   ~ 0
 RX
-Text Label 4050 2200 2    50   ~ 0
+Text Label 4050 3000 2    50   ~ 0
 GNSS_EN
 $Comp
@@
 L power:GND #PWR012
 U 1 1 5BC58E50
-P 3400 3000
-F 0 "#PWR012" H 3400 2750 50  0001 C CNN
-F 1 "GND" V 3405 2872 50  0000 R CNN
-F 2 "" H 3400 3000 50  0001 C CNN
-F 3 "" H 3400 3000 50  0001 C CNN
-	1    3400 3000
+P 3400 2700
+F 0 "#PWR012" H 3400 2450 50  0001 C CNN
+F 1 "GND" V 3405 2572 50  0000 R CNN
+F 2 "" H 3400 2700 50  0001 C CNN
+F 3 "" H 3400 2700 50  0001 C CNN
+	1    3400 2700
 	0    -1   -1   0
 $EndComp
@@
 	0    -1   -1   0
 $EndComp
-$Comp
-L power:GND #PWR09
-U 1 1 5B8876BC
-P 3400 2700
-F 0 "#PWR09" H 3400 2450 50  0001 C CNN
-F 1 "GND" V 3405 2572 50  0000 R CNN
-F 2 "" H 3400 2700 50  0001 C CNN
-F 3 "" H 3400 2700 50  0001 C CNN
-	1    3400 2700
-	0    -1   -1   0
-$EndComp
 Wire Wire Line
 	1950 5150 2800 5150
@@
 	5800 3550 5800 3650
 $Comp
-L power:GND #PWR024
+L power:GND #PWR013
 U 1 1 5BA03A7E
 P 7450 2400
-F 0 "#PWR024" H 7450 2150 50  0001 C CNN
+F 0 "#PWR013" H 7450 2150 50  0001 C CNN
 F 1 "GND" H 7455 2227 50  0000 C CNN
 F 2 "" H 7450 2400 50  0001 C CNN
@@
 VDD_GNSS
 $Comp
-L power:GNDD #PWR013
-U 1 1 5BA24559
-P 10650 6400
-F 0 "#PWR013" H 10650 6150 50  0001 C CNN
-F 1 "GNDD" H 10654 6245 50  0000 C CNN
-F 2 "" H 10650 6400 50  0001 C CNN
-F 3 "" H 10650 6400 50  0001 C CNN
-	1    10650 6400
-	0    1    1    0
-$EndComp
-$Comp
-L power:GND #PWR023
-U 1 1 5BA24653
-P 10950 6400
-F 0 "#PWR023" H 10950 6150 50  0001 C CNN
-F 1 "GND" H 10955 6227 50  0000 C CNN
-F 2 "" H 10950 6400 50  0001 C CNN
-F 3 "" H 10950 6400 50  0001 C CNN
-	1    10950 6400
-	0    -1   -1   0
-$EndComp
-$Comp
-L Device:R R7
-U 1 1 5BA6FAC8
-P 10800 6400
-F 0 "R7" V 10593 6400 50  0000 C CNN
-F 1 "0" V 10684 6400 50  0000 C CNN
-F 2 "Resistor_SMD:R_0603_1608Metric" V 10730 6400 50  0001 C CNN
-F 3 "~" H 10800 6400 50  0001 C CNN
-	1    10800 6400
-	0    1    1    0
-$EndComp
+L Device:R R5
+U 1 1 5BA46EC6
+P 7950 4050
+F 0 "R5" H 8020 4096 50  0000 L CNN
+F 1 "1M" H 8020 4005 50  0000 L CNN
+F 2 "Resistor_SMD:R_0603_1608Metric" V 7880 4050 50  0001 C CNN
+F 3 "~" H 7950 4050 50  0001 C CNN
+	1    7950 4050
+	1    0    0    -1
+$EndComp
+Wire Wire Line
+	8450 4100 8450 4200
+Text Label 7550 3900 0    50   ~ 0
+DISP_EN
+Wire Wire Line
+	7550 3900 7950 3900
+Connection ~ 7950 3900
+Wire Wire Line
+	7950 3900 8150 3900
+Text GLabel 8450 4300 2    50   Input ~ 0
+3V
+$Comp
+L Device:Q_PMOS_GSD Q2
+U 1 1 5BA46ED3
+P 8350 3900
+F 0 "Q2" H 8556 3946 50  0000 L CNN
+F 1 "SI2333DS-T1-E3" H 8556 3855 50  0000 L CNN
+F 2 "Package_TO_SOT_SMD:SOT-23" H 8550 4000 50  0001 C CNN
+F 3 "https://www.vishay.com/docs/72023/72023.pdf" H 8350 3900 50  0001 C CNN
+	1    8350 3900
+	1    0    0    -1
+$EndComp
+Wire Wire Line
+	7950 4200 8450 4200
+Connection ~ 8450 4200
+Wire Wire Line
+	8450 4200 8450 4300
+Wire Wire Line
+	8450 3700 8450 3500
+Text Label 8450 3500 0    50   ~ 0
+VDD_DISP
+Text Label 10200 2350 0    50   ~ 0
+VDD_DISP
+Wire Wire Line
+	10200 2250 10650 2250
+Wire Wire Line
+	10200 2350 10650 2350
+Wire Wire Line
+	10650 2250 10650 2350
+Connection ~ 10650 2250
+Connection ~ 10650 2350
+Text Label 4050 2200 2    50   ~ 0
+DISP_EN
+Wire Wire Line
+	4050 3000 3400 3000
 $EndSCHEMATC
